File: Coco2Composite.sch (EAGLE design)
At the start: 20 parts, among them J1 TO_COCO2, J2-SND RCA, J3-COMPOSITE RCA, Q1 BC557, Q2 BC547, U1 MC1372

Commit message: v1.1 revision
Parts:
- removed D1-1N4001: 1N4004, diode:1N4004
- removed J2-SND, J3-COMPOSITE: RCA, SparkFun-Connectors:RCA
- removed JP1: COMPOSITE_OUT, jumper:JP1E
- removed JP2: SOUND_OUT, jumper:JP1E
- added D1: 1N4004, diode:1N4004
- added J2: JACK_CONN1, SparkFun-Connectors:CONN_14
- added J3: JACK_CONN2, SparkFun-Connectors:CONN_14
- added J4: JACK_CONN3, SparkFun-Connectors:CONN_14
- added J5: JACK_CONN4, SparkFun-Connectors:CONN_14
- added J6: OUT_JACK, SparkFun-Connectors:CONN_03
Connections:
- net GND: now also J6.2; no longer JP1.1, JP2.1
- net N$1: now also D1.C, U1.RF_TANK_1; no longer D1-1N4001.C, U1.RF_TANK_2
- net N$10: now also J6.3; no longer JP2.2
- net N$2: now also D1.A, U1.RF_TANK_2; no longer D1-1N4001.A, U1.RF_TANK_1
- net N$9: now also J6.1; no longer JP1.2
Other:
- moved on the sheet: R1
